File: beginner_led_pcb.kicad_pcb (KiCad board)
At the start: 2 copper layers, 58.5 x 14.5 mm, 30 parts, among them J1 Conn_01x03_Pin

Commit message: gerber files
Routing:
- net +5V: track 81.1 -> 78.9 mm
Changed lines of the file:
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@@
   (segment (start 212.175 111.395) (end 212.175 113.035) (width 0.8) (layer "F.Cu") (net 1))
   (segment (start 216.225 113.045) (end 216.23 113.05) (width 0.8) (layer "F.Cu") (net 1))
+  (segment (start 213.65 111.495) (end 212.225 111.495) (width 1) (layer "F.Cu") (net 1))
+  (segment (start 208.225 111.495) (end 208.125 111.395) (width 1) (layer "F.Cu") (net 1))
   (segment (start 228.375 111.395) (end 228.375 113.045) (width 0.8) (layer "F.Cu") (net 1))
   (segment (start 208.125 111.395) (end 208.13 111.4) (width 1) (layer "F.Cu") (net 1))
+  (segment (start 240.575 111.495) (end 240.525 111.445) (width 1) (layer "F.Cu") (net 1))
   (segment (start 240.525 111.395) (end 240.525 113.045) (width 0.8) (layer "F.Cu") (net 1))
-  (segment (start 249.37 113.05) (end 250.17 113.05) (width 1) (layer "F.Cu") (net 1))
-  (segment (start 229.85 111.495) (end 229.85 113.04) (width 0.8) (layer "F.Cu") (net 1))
+  (segment (start 228.425 111.495) (end 228.375 111.445) (width 1) (layer "F.Cu") (net 1))
   (segment (start 225.81 113.05) (end 228.37 113.05) (width 1) (layer "F.Cu") (net 1))
-  (segment (start 237.95 111.495) (end 237.95 113.03) (width 0.8) (layer "F.Cu") (net 1))
+  (segment (start 212.225 111.495) (end 212.175 111.445) (width 1) (layer "F.Cu") (net 1))
+  (segment (start 248.7 111.495) (end 248.65 111.445) (width 1) (layer "F.Cu") (net 1))
   (segment (start 232.425 111.395) (end 232.425 113.045) (width 0.8) (layer "F.Cu") (net 1))
   (segment (start 224.325 113.025) (end 224.35 113.05) (width 0.8) (layer "F.Cu") (net 1))
+  (segment (start 229.85 111.495) (end 228.425 111.495) (width 1) (layer "F.Cu") (net 1))
   (segment (start 213.65 113.05) (end 216.23 113.05) (width 1) (layer "F.Cu") (net 1))
   (segment (start 232.42 113.05) (end 233.88 113.05) (width 1) (layer "F.Cu") (net 1))
   (segment (start 240.53 113.05) (end 242 113.05) (width 1) (layer "F.Cu") (net 1))
-  (segment (start 209.6 111.495) (end 209.6 113.05) (width 0.8) (layer "F.Cu") (net 1))
-  (segment (start 221.75 111.495) (end 221.75 113.04) (width 0.8) (layer "F.Cu") (net 1))
-  (segment (start 233.9 113.03) (end 233.88 113.05) (width 0.8) (layer "F.Cu") (net 1))
-  (segment (start 246.05 111.495) (end 246.05 113.04) (width 0.8) (layer "F.Cu") (net 1))
+  (segment (start 217.7 111.495) (end 216.275 111.495) (width 1) (layer "F.Cu") (net 1))
   (segment (start 208.12 111.4) (end 208.125 111.395) (width 1) (layer "F.Cu") (net 1))
   (segment (start 229.86 113.05) (end 232.42 113.05) (width 1) (layer "F.Cu") (net 1))
-  (segment (start 242 111.495) (end 242 113.05) (width 0.8) (layer "F.Cu") (net 1))
-  (segment (start 221.75 113.04) (end 221.74 113.05) (width 0.8) (layer "F.Cu") (net 1))
-  (segment (start 250.125 111.495) (end 250.125 113.005) (width 0.8) (layer "F.Cu") (net 1))
-  (segment (start 217.7 111.495) (end 217.7 113.05) (width 0.8) (layer "F.Cu") (net 1))
+  (segment (start 242 111.495) (end 240.575 111.495) (width 1) (layer "F.Cu") (net 1))
+  (segment (start 237.95 111.495) (end 236.525 111.495) (width 1) (layer "F.Cu") (net 1))
   (segment (start 236.475 113.045) (end 236.47 113.05) (width 0.8) (layer "F.Cu") (net 1))
+  (segment (start 232.475 111.495) (end 232.425 111.445) (width 1) (layer "F.Cu") (net 1))
   (segment (start 232.425 113.045) (end 232.42 113.05) (width 0.8) (layer "F.Cu") (net 1))
   (segment (start 208.13 113.05) (end 209.6 113.05) (width 1) (layer "F.Cu") (net 1))
-  (segment (start 237.95 113.03) (end 237.97 113.05) (width 0.8) (layer "F.Cu") (net 1))
   (segment (start 228.37 113.05) (end 229.86 113.05) (width 1) (layer "F.Cu") (net 1))
   (segment (start 236.47 113.05) (end 237.97 113.05) (width 1) (layer "F.Cu") (net 1))
+  (segment (start 221.75 111.495) (end 220.325 111.495) (width 1) (layer "F.Cu") (net 1))
   (segment (start 236.475 111.395) (end 236.475 113.045) (width 0.8) (layer "F.Cu") (net 1))
   (segment (start 206 111.4) (end 208.12 111.4) (width 1) (layer "F.Cu") (net 1))
+  (segment (start 244.625 111.495) (end 244.575 111.445) (width 1) (layer "F.Cu") (net 1))
   (segment (start 240.525 113.045) (end 240.53 113.05) (width 0.8) (layer "F.Cu") (net 1))
   (segment (start 220.275 113.045) (end 220.28 113.05) (width 0.8) (layer "F.Cu") (net 1))
-  (segment (start 225.8 113.04) (end 225.81 113.05) (width 0.8) (layer "F.Cu") (net 1))
   (segment (start 248.65 111.395) (end 248.65 113.04) (width 0.8) (layer "F.Cu") (net 1))
   (segment (start 221.74 113.05) (end 224.35 113.05) (width 1) (layer "F.Cu") (net 1))
-  (segment (start 250.125 113.005) (end 250.17 113.05) (width 0.8) (layer "F.Cu") (net 1))
   (segment (start 228.375 113.045) (end 228.37 113.05) (width 0.8) (layer "F.Cu") (net 1))
   (segment (start 248.65 113.04) (end 248.64 113.05) (width 0.8) (layer "F.Cu") (net 1))
+  (segment (start 220.325 111.495) (end 220.275 111.445) (width 1) (layer "F.Cu") (net 1))
   (segment (start 246.06 113.05) (end 248.64 113.05) (width 1) (layer "F.Cu") (net 1))
+  (segment (start 250.125 111.495) (end 248.7 111.495) (width 1) (layer "F.Cu") (net 1))
   (segment (start 212.16 113.05) (end 213.65 113.05) (width 1) (layer "F.Cu") (net 1))
   (segment (start 216.23 113.05) (end 217.7 113.05) (width 1) (layer "F.Cu") (net 1))
+  (segment (start 209.6 111.495) (end 208.225 111.495) (width 1) (layer "F.Cu") (net 1))
   (segment (start 204.53 111.29) (end 205.89 111.29) (width 1) (layer "F.Cu") (net 1))
+  (segment (start 224.375 111.495) (end 224.325 111.445) (width 1) (layer "F.Cu") (net 1))
+  (segment (start 216.275 111.495) (end 216.225 111.445) (width 1) (layer "F.Cu") (net 1))
   (segment (start 244.575 111.395) (end 244.575 113.035) (width 0.8) (layer "F.Cu") (net 1))
+  (segment (start 246.05 111.495) (end 244.625 111.495) (width 1) (layer "F.Cu") (net 1))
   (segment (start 242 113.05) (end 244.59 113.05) (width 1) (layer "F.Cu") (net 1))
   (segment (start 244.59 113.05) (end 246.06 113.05) (width 1) (layer "F.Cu") (net 1))
-  (segment (start 229.85 113.04) (end 229.86 113.05) (width 0.8) (layer "F.Cu") (net 1))
-  (segment (start 233.9 111.495) (end 233.9 113.03) (width 0.8) (layer "F.Cu") (net 1))
   (segment (start 224.325 111.395) (end 224.325 113.025) (width 0.8) (layer "F.Cu") (net 1))
-  (segment (start 213.65 111.495) (end 213.65 113.05) (width 0.8) (layer "F.Cu") (net 1))
+  (segment (start 236.525 111.495) (end 236.475 111.445) (width 1) (layer "F.Cu") (net 1))
   (segment (start 209.6 113.05) (end 212.16 113.05) (width 1) (layer "F.Cu") (net 1))
-  (segment (start 248.64 113.05) (end 249.37 113.05) (width 1) (layer "F.Cu") (net 1))
   (segment (start 233.88 113.05) (end 236.47 113.05) (width 1) (layer "F.Cu") (net 1))
-  (segment (start 225.8 111.495) (end 225.8 113.04) (width 0.8) (layer "F.Cu") (net 1))
   (segment (start 224.35 113.05) (end 225.81 113.05) (width 1) (layer "F.Cu") (net 1))
   (segment (start 237.97 113.05) (end 240.53 113.05) (width 1) (layer "F.Cu") (net 1))
@@
   (segment (start 212.175 113.035) (end 212.16 113.05) (width 0.8) (layer "F.Cu") (net 1))
   (segment (start 217.7 113.05) (end 220.28 113.05) (width 1) (layer "F.Cu") (net 1))
-  (segment (start 246.05 113.04) (end 246.06 113.05) (width 0.8) (layer "F.Cu") (net 1))
   (segment (start 244.575 113.035) (end 244.59 113.05) (width 0.8) (layer "F.Cu") (net 1))
+  (segment (start 233.9 111.495) (end 232.475 111.495) (width 1) (layer "F.Cu") (net 1))
+  (segment (start 225.8 111.495) (end 224.375 111.495) (width 1) (layer "F.Cu") (net 1))
   (segment (start 222.85 108.4625) (end 222.8625 108.45) (width 0.8) (layer "F.Cu") (net 2))
   (segment (start 203.805 110.04) (end 202.94 110.04) (width 0.4) (layer "F.Cu") (net 2))

Commit message: new components
Parts:
- removed D12, D13: D_TVS, Diode_SMD:D_SOD-323
- removed R2: 430R, Resistor_SMD:R_0603_1608Metric
- C1, C10, C11, C2, C3, C4, C5, C6, C7, C8, C9: footprint Capacitor_SMD:C_0603_1608Metric -> Capacitor_SMD:C_0402_1005Metric
- FB1: footprint Inductor_SMD:L_0603_1608Metric -> Inductor_SMD:L_0805_2012Metric
- R1: value 330R -> 1k0
- moved PWR 3.07 mm to (203.5, 107.1), turned to 180 degrees
- moved R1 2.77 mm to (203.5, 108.3), turned to 180 degrees
- moved C2 2.15 mm to (210.0, 110.7)
- moved C11 2.14 mm to (246.5, 110.7)
- moved C7 2.14 mm to (230.3, 110.7)
- moved C3 2.14 mm to (214.1, 110.7)
- moved C5 2.14 mm to (222.2, 110.7)
- moved C6 2.14 mm to (226.2, 110.7)
- moved C8 2.14 mm to (234.3, 110.7)
- moved D1 2.14 mm to (208.0, 110.6), turned to 180 degrees
- moved D11 2.14 mm to (248.5, 110.6), turned to 180 degrees
- moved D4 2.14 mm to (220.2, 110.6), turned to 180 degrees
- moved D6 2.14 mm to (228.3, 110.6), turned to 180 degrees
- moved D2 2.14 mm to (212.1, 110.6), turned to 180 degrees
- moved D5 2.14 mm to (224.2, 110.6), turned to 180 degrees
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Connections:
- C12 pad 1: Net-(D12-A2) -> GND
- C12 pad 2: GND -> Net-(J1-Pin_1)
- D1 pad 1: +5V -> Net-(D1-DOUT)
- D1 pad 2: Net-(D1-DOUT) -> GND
- D1 pad 3: GND -> D0
- D1 pad 4: D0 -> +5V
- D10 pad 1: +5V -> Net-(D10-DOUT)
- D10 pad 2: Net-(D10-DOUT) -> GND
- D10 pad 3: GND -> Net-(D10-DIN)
- D10 pad 4: Net-(D10-DIN) -> +5V
- D11 pad 1: +5V -> /NeoPixels 1|11/DOUT
- D11 pad 2: /NeoPixels 1|11/DOUT -> GND
- D11 pad 3: GND -> Net-(D10-DOUT)
- D11 pad 4: Net-(D10-DOUT) -> +5V
- D2 pad 1: +5V -> Net-(D2-DOUT)
- D2 pad 2: Net-(D2-DOUT) -> GND
- D2 pad 3: GND -> Net-(D1-DOUT)
- D2 pad 4: Net-(D1-DOUT) -> +5V
- D3 pad 1: +5V -> Net-(D3-DOUT)
- D3 pad 2: Net-(D3-DOUT) -> GND
- D3 pad 3: GND -> Net-(D2-DOUT)
- D3 pad 4: Net-(D2-DOUT) -> +5V
- D4 pad 1: +5V -> Net-(D4-DOUT)
- D4 pad 2: Net-(D4-DOUT) -> GND
- D4 pad 3: GND -> Net-(D3-DOUT)
- D4 pad 4: Net-(D3-DOUT) -> +5V
- D5 pad 1: +5V -> Net-(D5-DOUT)
- D5 pad 2: Net-(D5-DOUT) -> GND
- D5 pad 3: GND -> Net-(D4-DOUT)
- D5 pad 4: Net-(D4-DOUT) -> +5V
- D6 pad 1: +5V -> Net-(D6-DOUT)
- D6 pad 2: Net-(D6-DOUT) -> GND
- D6 pad 3: GND -> Net-(D5-DOUT)
- D6 pad 4: Net-(D5-DOUT) -> +5V
- D7 pad 1: +5V -> Net-(D7-DOUT)
- D7 pad 2: Net-(D7-DOUT) -> GND
- D7 pad 3: GND -> Net-(D6-DOUT)
- D7 pad 4: Net-(D6-DOUT) -> +5V
- D8 pad 1: +5V -> Net-(D8-DOUT)
- D8 pad 2: Net-(D8-DOUT) -> GND
- D8 pad 3: GND -> Net-(D7-DOUT)
- D8 pad 4: Net-(D7-DOUT) -> +5V
- D9 pad 1: +5V -> Net-(D10-DIN)
- D9 pad 2: Net-(D10-DIN) -> GND
- D9 pad 3: GND -> Net-(D8-DOUT)
- D9 pad 4: Net-(D8-DOUT) -> +5V
- FB1 pad 1: Net-(D12-A2) -> Net-(J1-Pin_1)
- J1 pad 1: Net-(D12-A2) -> Net-(J1-Pin_1)
- J1 pad 2: Net-(D13-A2) -> D0
- R1 pad 1: Net-(D13-A2) -> +5V
- R1 pad 2: D0 -> Net-(D14-A)
Routing:
- net +5V: track 78.9 -> 58.3 mm
- net Net-(D13-A2): track 8.42 -> 0.00 mm
- net Net-(D12-A2): track 7.84 -> 0.00 mm
- net Net-(J1-Pin_1): track 0.00 -> 5.97 mm
- net GND: track 35.9 -> 31.0 mm, vias 25 -> 34
- net D0: track 5.85 -> 10.2 mm, vias 0 -> 2
- net Net-(D10-DIN): track 3.71 -> 7.10 mm
- net Net-(D4-DOUT): track 3.71 -> 7.09 mm
- net Net-(D2-DOUT): track 3.71 -> 7.02 mm
- net Net-(D3-DOUT): track 3.71 -> 7.02 mm
- net Net-(D5-DOUT): track 3.71 -> 7.01 mm
- net Net-(D8-DOUT): track 3.71 -> 6.82 mm
- net Net-(D10-DOUT): track 3.73 -> 6.84 mm
- net Net-(D6-DOUT): track 3.71 -> 6.81 mm
- net Net-(D1-DOUT): track 3.71 -> 6.81 mm
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- added copper zone on F.Cu, net GND
Other:
- board size 58.5 x 14.5 mm -> 58 x 14.5 mm
- board text added: "2023.09.25"
- board text added: "JLCJLCJLCJLC"
