File: neopixels_array.kicad_sch (KiCad schematic)
At the start: 22 parts

Commit message: new components
Parts:
- removed C? (x10): 100n, Capacitor_SMD:C_0603_1608Metric, symbol Device:C
- removed D? (x10): WS2812B, LED_SMD:LED_WS2812B-2020_PLCC4_2.0x2.0mm, symbol LED:WS2812B
- added C? (x10): 100n, Capacitor_SMD:C_0402_1005Metric, symbol Device:C
- added D? (x10): WS2812B, LED_SMD:LED_WS2812B-2020_PLCC4_2.0x2.0mm, symbol LED:WS2812B
- C?: footprint Capacitor_SMD:C_0603_1608Metric -> Capacitor_SMD:C_0402_1005Metric; JLCPCB Part # (none) -> C126527
- D?: JLCPCB Part # (none) -> C965555
Connections:
- net DIN: now also D?.3 (DIN); no longer D?.4 (DIN)
- net DOUT: now also D?.1 (DOUT)
- net VDD: now also D?.4 (VDD), C?.1, C?.1, C?.1, C?.1, C?.1, C?.1, C?.1, C?.1, C?.1, C?.1, D?.4 (VDD), D?.4 (VDD), D?.4 (VDD), D?.4 (VDD), D?.4 (VDD), D?.4 (VDD), D?.4 (VDD), D?.4 (VDD), D?.4 (VDD), D?.4 (VDD); no longer D?.1 (VDD)
- net VSS: now also D?.2 (VSS), C?.2, C?.2, C?.2, C?.2, C?.2, C?.2, C?.2, C?.2, C?.2, C?.2, D?.2 (VSS), D?.2 (VSS), D?.2 (VSS), D?.2 (VSS), D?.2 (VSS), D?.2 (VSS), D?.2 (VSS), D?.2 (VSS), D?.2 (VSS), D?.2 (VSS); no longer D?.3 (VSS)
- new net: D?.1 (DOUT), D?.3 (DIN) (x10)
